Commit message: adding planning for avoiding the sensor

File: bubble_force_estimation/urdf/ftsensor_fake.urdf.xacro (robot description, xacro)
@@ -1,5 +1,6 @@
 <?xml version="1.0"?>
 <robot name="ftsensor_mount" xmlns:xacro="http://www.ros.org/wiki/xacro">
-    <xacro:include filename="$(find bubble_force_estimation)/urdf/ftsensor.urdf.xacro"/>
+<!--    <xacro:include filename="$(find bubble_force_estimation)/urdf/ftsensor.urdf.xacro"/>-->
+    <xacro:include filename="$(find bubble_force_estimation)/urdf/ftsensor_tag_origin.urdf.xacro"/>
     <xacro:ftsensor_xacro/>
 </robot>

File: bubble_force_estimation/urdf/ftsensor_tag_origin.urdf.xacro (robot description, xacro)
@@ -7,4 +7,42 @@
     <xacro:property name="tool_value" value="$(arg tool_name)"/>
     <xacro:macro name="ftsensor_xacro">
+        <!-- APRIL TAG FRAME NAME -->
+        <link name="$(arg tag_name)">
+        </link>
+        <joint name="$(arg sensor_name)_tag_fake_joint" type="fixed">
+          <origin xyz="0.07577 0 0" rpy="0 0 0"/>
+          <parent link="$(arg tag_name)"/>
+          <child link="$(arg sensor_name)_support"/>
+        </joint>
+        <!-- FT Sensor Mounting Support -->
+        <link name="$(arg sensor_name)_support">
+          <inertial>
+            <mass value="0.0"/> <!-- This is not the true mass -->
+            <origin xyz="0 0 0"/>
+            <inertia ixx="1.0" ixy="0.0" ixz="0.0" iyy="1.0" iyz="0.0" izz="1.0"/> <!-- This are not the true inertia -->
+          </inertial>
+          <visual>
+            <origin rpy="3.1415 0 -1.96349" xyz="0.0 0 0"/>
+            <geometry>
+              <mesh filename="package://bubble_force_estimation/meshes/visual/ft_mount_with_tag_support.stl" scale=".001 .001 .001"/>
+            </geometry>
+            <material name="grey">
+              <color rgba="0.5 0.5 0.5 1"/>
+            </material>
+          </visual>
+          <collision>
+            <origin rpy="3.1415 0 -1.96349" xyz="0.0 0 0"/>
+            <geometry>
+              <mesh filename="package://bubble_force_estimation/meshes/collision/ft_mount_with_tag_support.stl" scale=".001 .001 .001"/>
+            </geometry>
+          </collision>
+        </link>
+        <joint name="$(arg sensor_name)_support_joint" type="fixed">
+            <!--  Choose one of this two configurations  -->
+            <origin xyz="0 0 0.028" rpy="0 0 -1.5707"/>
+<!--            <origin xyz="0 0 -0.028" rpy="0 0 -1.5707"/>-->
+            <parent link="$(arg sensor_name)_support"/>
+            <child link="$(arg sensor_name)_base"/>
+        </joint>
         <!-- Make a base link. -->
         <link name="$(arg sensor_name)_base" type="fixed">
@@ -43,34 +81,4 @@
           </collision>
         </link>
-        <joint name="$(arg sensor_name)_support_joint" type="fixed">
-            <!--  Choose one of this two configurations  -->
-            <origin xyz="0 0 -0.028" rpy="0 0 1.5707"/>
-<!--            <origin xyz="0 0 -0.028" rpy="0 0 -1.5707"/>-->
-            <parent link="$(arg sensor_name)_base"/>
-            <child link="$(arg sensor_name)_support"/>
-        </joint>
-        <!-- FT Sensor Mounting Support -->
-        <link name="$(arg sensor_name)_support">
-          <inertial>
-            <mass value="0.0"/> <!-- This is not the true mass -->
-            <origin xyz="0 0 0"/>
-            <inertia ixx="1.0" ixy="0.0" ixz="0.0" iyy="1.0" iyz="0.0" izz="1.0"/> <!-- This are not the true inertia -->
-          </inertial>
-          <visual>
-            <origin rpy="3.1415 0 -1.96349" xyz="0.0 0 0"/>
-            <geometry>
-              <mesh filename="package://bubble_force_estimation/meshes/visual/ft_mount_with_tag_support.stl" scale=".001 .001 .001"/>
-            </geometry>
-            <material name="grey">
-              <color rgba="0.5 0.5 0.5 1"/>
-            </material>
-          </visual>
-          <collision>
-            <origin rpy="3.1415 0 -1.96349" xyz="0.0 0 0"/>
-            <geometry>
-              <mesh filename="package://bubble_force_estimation/meshes/collision/ft_mount_with_tag_support.stl" scale=".001 .001 .001"/>
-            </geometry>
-          </collision>
-        </link>
         <joint name="$(arg sensor_name)_tool_joint" type="fixed">
             <origin xyz="0 0 0" rpy="0 0 0"/>
@@ -100,17 +108,4 @@
             </geometry>
           </collision>
-        </link>
-        <!-- APRIL TAG FRAME NAME -->
-        <joint name="$(arg sensor_name)_tag_fake_joint" type="fixed">
-          <origin xyz="-0.07577 0 0" rpy="0 0 -1.57079"/>
-          <parent link="$(arg sensor_name)_support"/>
-          <child link="$(arg tag_name)"/>
-        </joint>
-        <link name="$(arg tag_name)">
-          <inertial>
-            <mass value="0.0"/>
-            <origin xyz="0 0 0"/>
-            <inertia ixx="0.0" ixy="0.0" ixz="0.0" iyy="0.0" iyz="0.0" izz="0.0"/>
-          </inertial>
         </link>
         <!-- APRIL TOOL FRAME NAME -->
