Commit message: fixing the ture sensor orientation

File: bubble_force_estimation/urdf/ftsensor.urdf.xacro (robot description, xacro)
@@ -3,5 +3,5 @@
     <xacro:arg name="sensor_name" default="netft"/>
     <xacro:arg name="tag_name" default="tag_0"/>
-    <xacro:arg name="tool_name" default="r15mm_ati_cylinder"/> <!-- Other values: bubbles, bubbles_flipped -->
+    <xacro:arg name="tool_name" default="r7p5mm_ati_cylinder"/> <!-- Other values: bubbles, bubbles_flipped -->
     <xacro:property name="tool_value" value="$(arg tool_name)"/>
     <xacro:macro name="ftsensor_xacro">
@@ -43,5 +43,7 @@
         </link>
         <joint name="$(arg sensor_name)_support_joint" type="fixed">
-            <origin xyz="0 0 -0.028" rpy="0 0 0"/>
+            <!--  Choose one of this two configurations  -->
+            <origin xyz="0 0 -0.028" rpy="0 0 1.5707"/>
+<!--            <origin xyz="0 0 -0.028" rpy="0 0 -1.5707"/>-->
             <parent link="$(arg sensor_name)_base"/>
             <child link="$(arg sensor_name)_support"/>

Commit message: adding static rod

File: bubble_force_estimation/urdf/ftsensor.urdf.xacro (robot description, xacro)
@@ -9,8 +9,8 @@
         <!-- Make a base link. -->
         <link name="$(arg sensor_name)_base" type="fixed">
-            <inertial>
-                <mass value="0"/>
-                <inertia ixx="0"  ixy="0"  ixz="0" iyy="0" iyz="0" izz="0" />
-            </inertial>
+<!--            <inertial>-->
+<!--                <mass value="0"/>-->
+<!--                <inertia ixx="0"  ixy="0"  ixz="0" iyy="0" iyz="0" izz="0" />-->
+<!--            </inertial>-->
         </link>
         <joint name="$(arg sensor_name)_sensor_joint" type="fixed">

File: bubble_force_estimation/urdf/ftsensor_fake.urdf.xacro (robot description, xacro)
@@ -1,6 +1,6 @@
 <?xml version="1.0"?>
 <robot name="ftsensor_mount" xmlns:xacro="http://www.ros.org/wiki/xacro">
-<!--    <xacro:include filename="$(find bubble_force_estimation)/urdf/ftsensor.urdf.xacro"/>-->
-    <xacro:include filename="$(find bubble_force_estimation)/urdf/ftsensor_tag_origin.urdf.xacro"/>
+    <xacro:include filename="$(find bubble_force_estimation)/urdf/ftsensor.urdf.xacro"/>
+<!--    <xacro:include filename="$(find bubble_force_estimation)/urdf/ftsensor_tag_origin.urdf.xacro"/>-->
     <xacro:ftsensor_xacro/>
 </robot>
